File: PCB/RCONTROL/rcontrol.sch (EAGLE design)
At the start: 13 parts

Commit message: New PCB
New PCB
Parts:
- removed DD1: (no value), pepelac:PROC
- removed U$2: (no value), pinhead:PINHD-3X9
- removed U$3: LD333.3, lm1117:LD333.3
- added ANT: (no value), pinhead:PINHD-1X1
- added C4, C5: 22pF, rcl:C-EUC0805
- added IC1: LM1117IMPX-3.3, lm1117:LM1117IMPX-3.3
- added IC2: STM32F10XCXT6, STM32:STM32F10XCXT6
- added Q1: 8MHz, crystal:CRYSTALHC49U-V
- added U1: PINHD3X9, pinheader3x9:PINHD3X9
- C2: value 1uF -> 1uf; device SparkFun-Capacitors:10UF-16V-10%(TANT) -> rcl:CPOL-EUCT3528
- C3: device rcl:C-EUC1206 -> rcl:C-EUC0805
- renumbered LED1 to RED, LED2 to GREEN, U$1 to ESP8266
Connections:
- new net N$19: ESP8266.CH_PD, IC2PORTB_H.PB9
- new net N$36: C3.1, IC2RESET.NRST, S1.3, S1.4
- new net N$37: C5.1, IC2PORTD/OSC.PD1/OSC=>, Q1.2
- new net N$9: ANT.1, ESP8266.ANT
- net +3V3: now also IC1.OUT, IC1.OUT1, IC2AN_POWER.VDDA, IC2POWER.VDD_1, IC2POWER.VDD_2, IC2POWER.VDD_3; no longer DD1.VCC_A, ESP8266.CH_PD, U$3.OUT
- net GND: now also C4.2, C5.2, IC1.GND, IC2AN_POWER.VSSA, IC2POWER.VSS_1, IC2POWER.VSS_2, IC2POWER.VSS_3, SWD.2, U1.12, U1.15, U1.18, U1.21, U1.24, U1.27, U1.3, U1.6, U1.9; no longer DD1.GND_A, SWD.1, U$2.12, U$2.15, U$2.18, U$2.21, U$2.24, U$2.27, U$2.3, U$2.6, U$2.9, U$3.ADJ
- net N$1: now also IC2PORTA_L.PA0, U1.1; no longer DD1.PA9, ESP8266.RX
- net N$10: now also IC2PORTB_L.PB1, U1.22; no longer DD1.PA0, U$2.1
- net N$11: now also IC2PORTB_H.PB10, U1.25; no longer DD1.PA1, U$2.4
- net N$12: now also IC2PORTB_H.PB11, U1.26; no longer DD1.PA2, U$2.7
- net N$13: now also ESP8266.RX, IC2PORTA_H.PA9; no longer DD1.PA3, U$2.10
- net N$14: now also ESP8266.TX, IC2PORTA_H.PA10; no longer DD1.PA6, U$2.13
- net N$15: now also IC2PORTA_H.PA13, SWD.1; no longer DD1.PA7, U$2.16
- net N$16: now also IC2PORTA_H.PA14, SWD.3; no longer DD1.PB0, U$2.19
- net N$17: now also IC2PORTA_H.PA15, R1.2; no longer DD1.PB1, U$2.22
- net N$18: now also IC2PORTB_L.PB3, R2.2; no longer DD1.SDA, U$2.26
- net N$2: now also IC2PORTA_L.PA1, U1.4; no longer DD1.PA10, ESP8266.TX
- net N$23: now also IC1.IN, U1.11, U1.14, U1.17, U1.2, U1.20, U1.23, U1.5, U1.8; no longer U$2.11, U$2.14, U$2.17, U$2.2, U$2.20, U$2.23, U$2.5, U$2.8, U$3.IN
- net N$3: now also IC2PORTA_L.PA2, U1.7; no longer DD1.PA13, SWD.3
- net N$4: now also IC2PORTA_L.PA3, U1.10; no longer DD1.SCL, U$2.25
- net N$5: now also IC2PORTA_L.PA6, U1.13; no longer DD1.PA14, SWD.2
- net N$6: now also C4.1, IC2PORTD/OSC.PD0/OSC<=, Q1.1; no longer C3.1, DD1.RESET, S1.3, S1.4
- net N$7: now also IC2PORTA_L.PA7, U1.16; no longer DD1.PA15, R1.2
- net N$8: now also IC2PORTB_L.PB0, U1.19; no longer DD1.PB3, R2.2
Other:
- moved on the sheet: C2, C3, S1, SWD
