File: PCB/RCONTROL/rcontrolv0.1.brd (EAGLE design)
At the start: 25.7 x 42.9 mm, 17 parts, among them IC1 LM1117IMPX-3.3, Q1 8MHz, U1 PINHD3X9

Commit message: New PCB
New PCB
Parts:
- removed ANT: (no value), pinhead:1X01
- removed C4, C5: 22pF, rcl:C0805
- removed ESP8266: ESP8266_ESP-03, ESP8266:ESP-03
- removed Q1: 8MHz, crystal:HC49U-V
- removed U1: PINHD3X9, pinheader3x9:3X9
- added U$1: ESP8266_ESP-03, ESP8266:ESP-03
- added U$2: (no value), pinhead:3X09
- C2: value 1uf -> (none)
- C3: device rcl:C0805 -> rcl:C1206
- moved C2 70.1 mm to (-11.4, -31.8), flipped to the top
- moved IC1 54.9 mm to (-8.89, -22.9), flipped to the top, turned to 0 degrees
- moved RED 12.0 mm to (13.8, 5.41), turned to 90 degrees
- moved C1 9.70 mm to (23.5, 21.6), flipped to the top, turned to 180 degrees
- moved SWD 6.88 mm to (2.54, 24.1)
- moved DD1 4.55 mm to (10.7, 27.9)
- moved R1 4.40 mm to (9.12, 5.41), turned to 0 degrees
- moved R2 4.15 mm to (18.3, 5.38)
- moved GREEN 4.12 mm to (22.8, 5.38)
- moved C3 3.12 mm to (2.11, 15.8)
- moved S1 1.42 mm to (3.43, 8.99), turned to 90 degrees
Connections:
- removed net N$19: DD1.46, ESP8266.6
- removed net N$37: C5.1, DD1.6, Q1.2
- removed net N$6: C4.1, DD1.5, Q1.1
- removed net N$9: ANT.1, ESP8266.7
- new net N$34: DD1.20, U$1.6
- new net N$35: C2.+, IC1.2
- net +3V3: now also U$1.8; no longer C2.+, ESP8266.8, IC1.2
- net GND: now also U$1.1, U$1.12, U$2.021, U$2.12, U$2.15, U$2.18, U$2.24, U$2.27, U$2.3, U$2.6, U$2.9; no longer C4.2, C5.2, ESP8266.1, ESP8266.12, U1.12, U1.15, U1.18, U1.21, U1.24, U1.27, U1.3, U1.6, U1.9
- net N$1: now also U$1.4; no longer ESP8266.4
- net N$10: now also U$2.1; no longer U1.1
- net N$11: now also U$2.4; no longer U1.4
- net N$12: now also U$2.7; no longer U1.7
- net N$13: now also U$2.10; no longer U1.10
- net N$14: now also U$2.13; no longer U1.13
- net N$15: now also U$2.16; no longer U1.16
- net N$16: now also U$2.19; no longer U1.19
- net N$17: now also U$2.022; no longer U1.22
- net N$18: now also U$2.26; no longer U1.26
- net N$2: now also U$1.3; no longer ESP8266.3
- net N$23: now also U$2.020, U$2.023, U$2.11, U$2.14, U$2.17, U$2.2, U$2.5, U$2.8; no longer U1.11, U1.14, U1.17, U1.2, U1.20, U1.23, U1.5, U1.8
- net N$4: now also U$2.25; no longer U1.25
Routing:
- net N$28: track 0.00 -> 75.0 mm
- net N$29: track 0.00 -> 74.9 mm
- net N$33: track 0.00 -> 57.1 mm
- net N$32: track 0.00 -> 57.1 mm
- net N$31: track 0.00 -> 55.9 mm
- net N$30: track 0.00 -> 55.9 mm
- net N$2: track 42.7 -> 12.3 mm
- net +3V3: track 59.7 -> 31.0 mm, vias 4 -> 1
- net N$36: track 27.6 -> 5.08 mm, vias 1 -> 0
- net N$1: track 37.8 -> 15.4 mm
- net N$19: track 22.4 -> 1.27 mm, vias 1 -> 0
- net N$37: track 9.84 -> 0.00 mm
- net N$6: track 8.95 -> 0.00 mm
- net N$12: track 12.8 -> 8.57 mm
- net N$18: track 10.5 -> 14.7 mm
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Other:
- board size 25.7 x 42.9 mm -> 26.6 x 45.4 mm
- board text added: "29.04.2015"
- board text added: "DiGiua.com"
- board text removed: "2015"
- board text removed: "digiua.com"
